File: encoder_pcb.kicad_pcb (KiCad board)
At the start: 2 copper layers, 50 x 50 mm, 28 parts, among them IC1 LT1117IST-3.3, J1 POWER, J2 TTL PROG (JST), J3 LEFT ENCODER (JST), J4 RIGHT ENCODER (JST), J5 TTL PROG (HEADER), J6 LEFT ENCODER (HEADER), J7 RIGHT ENCODER (HEADER), U1 ESP32-WROOM-32U

Commit message: Correct C2 value
Parts:
- C2: value 10 uf -> 1 uf
Changed lines of the file:
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@@
       (effects (font (size 1 1) (thickness 0.15)))
     )
-    (fp_text value "10 uf" (at 0 1.85) (layer "F.Fab")
+    (fp_text value "1 uf" (at 0 1.85) (layer "F.Fab")
       (effects (font (size 1 1) (thickness 0.15)))
     )
