File: encoder_pcb.kicad_sch (KiCad schematic)
At the start: 26 parts, among them IC1 LT1117IST-3.3, J1 POWER, J2 TTL PROG (JST), J3 LEFT ENCODER (JST), J4 RIGHT ENCODER (JST), J5 TTL PROG (HEADER), J6 LEFT ENCODER (HEADER), J7 RIGHT ENCODER (HEADER), U1 ESP32-WROOM-32U

Commit message: Correct C2 value
Parts:
- C2: value 10 uf -> 1 uf
Changed lines of the file:
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@@
       (effects (font (size 1.27 1.27)) (justify left))
     )
-    (property "Value" "10 uf" (id 1) (at 54.61 35.5599 0)
+    (property "Value" "1 uf" (id 1) (at 54.61 35.5599 0)
       (effects (font (size 1.27 1.27)) (justify left))
     )
@@
     )
     (path "/d7ea977c-3cc7-4aeb-b591-cfe1f0cef32c"
-      (reference "C2") (unit 1) (value "10 uf") (footprint "Capacitor_SMD:C_1206_3216Metric_Pad1.33x1.80mm_HandSolder")
+      (reference "C2") (unit 1) (value "1 uf") (footprint "Capacitor_SMD:C_1206_3216Metric_Pad1.33x1.80mm_HandSolder")
     )
     (path "/db616132-8151-422d-8fb2-791935386c88"
